Commit message: Add dummy base_link
Signed-off-by: Shravan Deva <devashravan7@gmail.com>

File: chitrak_description/urdf/chitrak.xacro (robot description, xacro)
@@ -6,6 +6,7 @@
 <robot
   name="chitrak_description">
-  <link
-    name="base_link">
+  <link name="base_link"></link>
+  <link
+    name="torso_link">
     <inertial>
       <origin
@@ -28,22 +29,27 @@
       <geometry>
         <mesh
-          filename="package://chitrak_description/meshes/base_link.STL" />
-      </geometry>
-      <material
-        name="">
-        <color
-          rgba="0.752941176470588 0.752941176470588 0.752941176470588 1" />
-      </material>
-    </visual>
-    <collision>
-      <origin
-        xyz="0 0 0"
-        rpy="0 0 0" />
-      <geometry>
-        <mesh
-          filename="package://chitrak_description/meshes/base_link.STL" />
-      </geometry>
-    </collision>
-  </link>
+          filename="package://chitrak_description/meshes/torso_link.STL" />
+      </geometry>
+      <material
+        name="">
+        <color
+          rgba="0.752941176470588 0.752941176470588 0.752941176470588 1" />
+      </material>
+    </visual>
+    <collision>
+      <origin
+        xyz="0 0 0"
+        rpy="0 0 0" />
+      <geometry>
+        <mesh
+          filename="package://chitrak_description/meshes/torso_link.STL" />
+      </geometry>
+    </collision>
+  </link>
+  <joint name="torso_joint" type="fixed">
+    <origin xyz ="0 0 0" rpy="0 0 0"/>
+    <parent link="base_link"/>
+    <child link="torso_link"/>
+  </joint>
   <link
     name="fr_hip_link">
@@ -93,5 +99,5 @@
       rpy="0 0 0" />
     <parent
-      link="base_link" />
+      link="torso_link" />
     <child
       link="fr_hip_link" />
@@ -267,5 +273,5 @@
       rpy="0 0 0" />
     <parent
-      link="base_link" />
+      link="torso_link" />
     <child
       link="fl_hip_link" />
@@ -441,5 +447,5 @@
       rpy="0 0 0" />
     <parent
-      link="base_link" />
+      link="torso_link" />
     <child
       link="br_hip_link" />
@@ -615,5 +621,5 @@
       rpy="0 0 0" />
     <parent
-      link="base_link" />
+      link="torso_link" />
     <child
       link="bl_hip_link" />
